File: 1802-Mini-Super-Elf-Bus.kicad_pcb (KiCad board)
At the start: 2 copper layers, 100 x 100 mm, 55 parts, among them J1 Mount, J10 SLOT_2_CONFIG, J2 Mount, J3 Mount, J4 Mount, J5 1802/Mini Bus, J6 SLOT_1_CONFIG, J7 Super Elf Bus, J8 USB PWR, J9 Serial Port, U1 4049, U2 4023, U3 4001, U4 4071, U5 4011, U6 40245, U7 HI_MEM, U8 LO_MEM, U9 LM2940CT

Commit message: Rev B updates
Parts:
- removed the C4 at (130.2, 126.4)
- removed the U3 at (135.3, 103.5)
- removed the U8 at (162.6, 134.0)
- added U4: 4001, Package_DIP:DIP-14_W7.62mm_Socket, F.Cu at (135.3, 103.5)
- added U6: LO_MEM, Package_DIP:DIP-28_W15.24mm_Socket, F.Cu at (160.7, 134.0)
- moved C4 15.2 mm to (130.2, 95.9)
- moved D2 14.0 mm to (130.2, 80.6)
- moved C2 3.86 mm to (125.1, 100.3)
- moved C3 3.81 mm to (125.1, 87.6)
- moved U9 3.81 mm to (125.1, 96.5)
- moved JP3 3.24 mm to (120.0, 76.8)
- moved JP10 3.17 mm to (120.0, 131.4)
- moved JP11 3.17 mm to (120.0, 134.0)
- moved JP2 3.17 mm to (120.0, 71.8)
- moved JP8 3.17 mm to (120.0, 128.9)
- moved JP9 3.17 mm to (120.0, 126.4)
- moved R16 3.17 mm to (107.3, 134.0)
- moved R17 3.17 mm to (109.9, 123.8)
- moved R18 3.17 mm to (112.4, 134.0)
- moved U1 3.17 mm to (107.3, 118.7)
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- renumbered C5 to C4, C6 to C5, C7 to C6, C8 to C7, D2 to D1, D1 to D2, R12 to R11, R13 to R12, R14 to R13, R15 to R14, R16 to R15, R17 to R16, R18 to R17, R19 to R18, U5 to U2, U4 to U3, U2 to U5, U6 to U8
Connections:
- J7 pad 10: TPB -> TPA
- J7 pad 11: M -> MP
- J7 pad 12: G -> (no net)
- J7 pad 13: ~CLEAR -> (no net)
- J7 pad 14: A15 -> /A14
- J7 pad 15: /A13 -> /A12
- J7 pad 16: /A11 -> /A10
- J7 pad 17: /A9 -> /A8
- J7 pad 18: /A7 -> /A6
- J7 pad 19: /A5 -> /A4
- J7 pad 2: 10V1 -> 10V2
- J7 pad 20: /A3 -> /A2
- J7 pad 21: /A1 -> /A0
- J7 pad 22: /D7 -> /D6
- J7 pad 23: /D5 -> /D4
- J7 pad 24: /D3 -> /D2
- J7 pad 25: /D1 -> /D0
- J7 pad 27: 10V2 -> 10V1
- J7 pad 28: ~EF2 -> ~EF3
- J7 pad 29: N1 -> N0
- J7 pad 3: ~EF3 -> ~EF2
- J7 pad 30: Q -> N2
- J7 pad 31: SC0 -> SC1
- J7 pad 32: CLOCK -> ~MRD
- J7 pad 33: ~DMAOUT -> ~DMAIN
- J7 pad 34: ~INT -> ~MWR
- J7 pad 35: TPA -> TPB
- J7 pad 36: MP -> M
- J7 pad 37: (no net) -> G
- J7 pad 38: (no net) -> ~CLEAR
- J7 pad 39: /A14 -> A15
- J7 pad 4: N0 -> N1
- J7 pad 40: /A12 -> /A13
- J7 pad 41: /A10 -> /A11
- J7 pad 42: /A8 -> /A9
- J7 pad 43: /A6 -> /A7
- J7 pad 44: /A4 -> /A5
- J7 pad 45: /A2 -> /A3
- J7 pad 46: /A0 -> /A1
- J7 pad 47: /D6 -> /D7
- J7 pad 48: /D4 -> /D5
- J7 pad 49: /D2 -> /D3
- J7 pad 5: N2 -> Q
- J7 pad 50: /D0 -> /D1
- J7 pad 6: SC1 -> SC0
- J7 pad 7: ~MRD -> CLOCK
- J7 pad 8: ~DMAIN -> ~DMAOUT
- J7 pad 9: ~MWR -> ~INT
- J8 pad 2: (no net) -> Net-(J8-Pad2)
- J8 pad 3: (no net) -> Net-(J8-Pad3)
- J8 pad 4: (no net) -> Net-(J8-Pad4)
- J8 pad 5: (no net) -> GND
- JP2 pad 1: 10V2 -> 10V1
- JP2 pad 3: 10V1 -> 10V2
- U1 pad 7: A15 -> ~MRD
- U2 pad 12: Net-(U4-Pad11) -> Net-(U2-Pad12)
- U2 pad 2: Net-(U4-Pad3) -> Net-(U2-Pad2)
- U2 pad 4: ~CS_LO -> Net-(U2-Pad2)
- U2 pad 5: Net-(U3-Pad3) -> Net-(U1-Pad6)
- U2 pad 6: MEN -> A15
- U3 pad 1: ~MRD -> Net-(U2-Pad12)
- U3 pad 11: Net-(U4-Pad11) -> Net-(U2-Pad12)
- U3 pad 2: Net-(U1-Pad6) -> Net-(U3-Pad2)
- U3 pad 3: Net-(U4-Pad3) -> ~CS_LO
- U5 pad 1: SC1 -> VCC
Routing:
- net ~INT: track 119.4 -> 210.9 mm, vias 5 -> 4
- net /A11: track 86.0 -> 131.9 mm, vias 3 -> 4
- net /A8: track 86.6 -> 129.3 mm, vias 2 -> 3
- net /A9: track 87.6 -> 125.6 mm, vias 3 -> 4
- net Net-(J9-Pad4): track 75.9 -> 110.8 mm
- net /D4: track 43.0 -> 10.3 mm
- net Net-(U3-Pad3): track 32.6 -> 0.00 mm
- net /A10: track 95.9 -> 125.4 mm, vias 3 -> 4
- net N0: track 138.3 -> 167.3 mm, vias 3 -> 1
- net SC0: track 138.1 -> 166.8 mm, vias 3 -> 1
- net Net-(U2-Pad12): track 0.00 -> 28.4 mm, vias 0 -> 1
- net Q: track 144.5 -> 118.8 mm
- net N1: track 145.3 -> 170.7 mm, vias 3 -> 1
- net /D3: track 7.22 -> 27.7 mm
- net Net-(U3-Pad2): track 0.00 -> 20.3 mm, vias 0 -> 2
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Other:
- board text added: "A1"
- board text added: "A11"
- board text added: "A13"
- board text added: "A15"
- board text added: "A3"
- board text added: "A5"
- board text added: "A7"
- board text added: "A9"
- board text added: "D1"
- board text added: "D3"
- board text added: "D5"
- board text added: "D7"
- board text added: "G"
- board text added: "M"
- board text added: "N2"
- board text added: "Super Elf Bus rev B"
- board text removed: "A0"
- board text removed: "A10"
- board text removed: "A12"
- board text removed: "A14"
- board text removed: "A2"
- board text removed: "A4"
- board text removed: "A6"
- board text removed: "A8"
- board text removed: "CLOCK-"
- board text removed: "D0"
- board text removed: "D2"
- board text removed: "D4"
- board text removed: "D6"
- board text removed: "DMAOUT-"
- board text removed: "INT-"
- board text removed: "MP"
- board text removed: "N/C"
- board text removed: "N1"
- board text removed: "P/NP"
- board text removed: "S. ELF PWR"
- board text removed: "Super Elf Bus rev A"
